File: uefi2.kicad_sch (KiCad schematic)
At the start: 304 parts, among them J1 Conn_01x05, J10 Conn_01x05, J11 USB_B_Mini, J2 MiniFit, J3 VRIN1, J4 VRIN2, J5 AudioJack_THR, J6 VROUT1, J7 ETB, J8 PPS, J9 XH-8A, M1 Module-power12-0.2, M10 Module-sd-0.1, M11 Module-can-0.1, M12 Module-wbo-0.3, M13 Module-can-0.1, M2 Module-power5-0.2, M3 Module-knock-0.1, M4 Module-knock-0.1, M5 Module-vr-0.1, M6 Module-output-0.3, M7 Module-input-0.1, M8 Module-ign8-0.2, M9 Module-mcu144-0.6, P1 P, P2 P, P3 P, P4 P, P5 P, P6 P, Q1 NGD8201AN, Q10 AUIPS2041LTR, Q2 NGD8201AN, Q3 NGD8201AN, Q4 NGD8201AN, Q5 NGD8201AN, Q6 NGD8201AN, Q7 NGD8201AN, Q8 NGD8201AN, Q9 AUIPS2041LTR, SW1 Button_SPST, SW2 Button_SPST, U1 TLS115_SOIC, U2 TLS115_SON, U3 MCP6002-xSN, U4 L6205PD, U5 MPX4_MAP, U6 MPXA6115A, U7 LIS2DW12TR, U8 LPS25HB

Commit message: attempt 6
Parts:
- removed BT1: BATTERY_CR2032, Battery:BatteryHolder_Keystone_1060_1x2032, symbol art-electro-power:BATTERY_CR2032
- removed C1, C2: 1u, hellen-one-common:C0603, symbol hellen-one-common:Cap
- removed C10: 10nF, Capacitor_SMD:C_0402_1005Metric, symbol Device:C
- removed C11, C12, C13, C15, C18, C20, C5, C6, C7, C9: 10u, Capacitor_SMD:C_0603_1608Metric, symbol Device:C
- removed C14: 220nF, Capacitor_SMD:C_0402_1005Metric, symbol Device:C
- removed C16, C17, C19, C21, C23, C3, C4: 100nF, Capacitor_SMD:C_0402_1005Metric, symbol Device:C
- removed C22: 100n, hellen-one-common:C0603, symbol hellen-one-common:Cap
- removed C8: 5.6nF, Capacitor_SMD:C_0402_1005Metric, symbol Device:C
- removed D1, D2: B5819W, Diode_SMD:D_SOD-123, symbol Diode:1N4148WS
- removed D10, D12, D14, D16, D18, D20, D22, D37, D39, D8: LED-RED-0603, LED_SMD:LED_0603_1608Metric, symbol Device:LED
- removed D11, D13, D15, D17, D19, D21, D34, D36, D38, D40, D42, D7, D9: 1N4148WS, Diode_SMD:D_SOD-323, symbol Diode:1N4148WS
- removed D23, D24, D25, D26, D27, D28, D29, D30: LED-BLUE-0603, LED_SMD:LED_0603_1608Metric, symbol Device:LED
- removed D3, D4: 1N4148WS, Diode_SMD:D_SOD-323, symbol Device:D
- removed D31, D32, D33, D35: LED-GREEN-0603, LED_SMD:LED_0603_1608Metric, symbol Device:LED
- removed D41: LED-WHITE-0603, LED_SMD:LED_0603_1608Metric, symbol Device:LED
- removed D43: 1N4148WS, hellen-one-common:SOD-323, symbol hellen-one-common:1N4148WS
- removed D5, D6: B5819W, Diode_SMD:D_SOD-123, symbol hellen-one-common:1N4148WS
- removed F1, F2, F3, F4, F5, F6, F7, F8: 10A, hellen-one-common:36911600000, symbol hellen-one-common:Fuse-Pad-Pad
- removed G1, G2: PROTO_AREA, hellen-one-common:PROTO_AREA, symbol hellen-one-common:PROTO_AREA
- removed J1: Conn_01x05, Connector_PinHeader_2.54mm:PinHeader_1x05_P2.54mm_Vertical, symbol Connector_Generic:Conn_01x05
- removed J10: Conn_01x05, Connector_PinHeader_2.00mm:PinHeader_1x05_P2.00mm_Vertical, symbol Connector_Generic:Conn_01x05
- removed J11: USB_B_Mini, hellen-one-common:USB-MINI-B-VERTICAL, symbol hellen-one-common:USB_B_Mini
- removed J2: MiniFit, Connector_Molex:Molex_Mini-Fit_Jr_5569-02A2_2x01_P4.20mm_Horizontal, symbol Connector_Generic:Conn_01x02
- removed J3: VRIN1, Connector_PinHeader_1.00mm:PinHeader_1x01_P1.00mm_Vertical, symbol Connector_Generic:Conn_01x01
- removed J4: VRIN2, Connector_PinHeader_1.00mm:PinHeader_1x01_P1.00mm_Vertical, symbol Connector_Generic:Conn_01x01
- removed J5: AudioJack_THR, hellen-one-common:Jack_3.5mm_PJ-3250-5A, symbol hellen-one-common:AudioJack_THR
- removed J6: VROUT1, Connector_PinHeader_1.00mm:PinHeader_1x01_P1.00mm_Vertical, symbol Connector_Generic:Conn_01x01
- removed J7: ETB, Connector_PinHeader_2.54mm:PinHeader_1x06_P2.54mm_Vertical, symbol Connector_Generic:Conn_01x06
- removed J8: PPS, Connector_PinHeader_2.54mm:PinHeader_1x04_P2.54mm_Vertical, symbol Connector_Generic:Conn_01x04
- removed J9: XH-8A, kicad6:XH-8A, symbol Connector_Generic:Conn_01x08
- removed JP1, JP10, JP11, JP12, JP13, JP14, JP15, JP16, JP17, JP18, JP19, JP2, JP20, JP21, JP22, JP23, JP24, JP25, JP28, JP29, JP3, JP30, JP31, JP32, JP33, JP34, JP35, JP4, JP5, JP6, JP7, JP8, JP9: Jumper_2_Open, hellen-one-common:PAD-0805-PAD, symbol hellen-one-common:Jumper-Pad-Pad
- removed JP26, JP27: Jumper_2_Open, hellen-one-common:PAD-1206-PAD, symbol hellen-one-common:Fuse-Pad-Pad
- removed KNOCK_RAW1: IN_KNOCK1_RAW, Connector_PinHeader_1.00mm:PinHeader_1x01_P1.00mm_Vertical, symbol Connector_Generic:Conn_01x01
- removed KNOCK_RAW2: IN_KNOCK2_RAW, Connector_PinHeader_1.00mm:PinHeader_1x01_P1.00mm_Vertical, symbol Connector_Generic:Conn_01x01
- removed M1: Module-power12-0.2, hellen-one-power12-0.2:power12, symbol power12-0.2:Module-power12-0.2
- removed M10: Module-sd-0.1, hellen-one-sd-0.1:sd, symbol sd-0.1:Module-sd-0.1
- removed M11, M13: Module-can-0.1, hellen-one-can-0.1:can, symbol can-0.1:Module-can-0.1
- removed M12: Module-wbo-0.3, hellen-one-wbo-0.3:wbo, symbol wbo-0.3:Module-wbo-0.3
- removed M2: Module-power5-0.2, hellen-one-power5-0.2:power5, symbol power5-0.2:Module-power5-0.2
- removed M3, M4: Module-knock-0.1, hellen-one-knock-0.1:knock, symbol knock-0.1:Module-knock-0.1
- removed M5: Module-vr-0.1, hellen-one-vr-0.1:vr, symbol hellen-one-vr-0.1:Module-vr-0.1
- removed M6: Module-output-0.3, hellen-one-output-0.3:output, symbol output-0.3:Module-output-0.3
- removed M7: Module-input-0.1, hellen-one-input-0.1:input, symbol input-0.1:Module-input-0.1
- removed M8: Module-ign8-0.2, hellen-one-ign8-0.2:ign8, symbol ign8-0.2:Module-ign8-0.2
- removed M9: Module-mcu144-0.6, hellen-one-mcu-0.6:mcu, symbol mcu-0.6:Module-mcu-0.6
- removed MMCU1, MMCU10, MMCU11, MMCU12, MMCU13, MMCU14, MMCU15, MMCU16, MMCU17, MMCU18, MMCU19, MMCU2, MMCU20, MMCU21, MMCU22, MMCU23, MMCU24, MMCU25, MMCU26, MMCU27, MMCU28, MMCU29, MMCU3, MMCU30, MMCU31, MMCU4, MMCU5, MMCU6, MMCU7, MMCU8, MMCU9: MMCU, Connector_PinHeader_1.00mm:PinHeader_1x01_P1.00mm_Vertical, symbol Connector_Generic:Conn_01x01
- removed P1, P2, P3, P4, P5, P6: P, Connector_Pin:Pin_D1.0mm_L10.0mm, symbol Connector_Generic:Conn_01x01
- removed PP1: Motronic_88pin, rusefi_lib_private:88pin_STS, symbol motronic_88pin_STS:Motronic_88pin
- removed Q1, Q2, Q3, Q4, Q5, Q6, Q7, Q8: NGD8201AN, Package_TO_SOT_SMD:TO-252-2, symbol Device:Q_NIGBT_GCE
- removed Q10, Q9: AUIPS2041LTR, Package_TO_SOT_SMD:SOT-223, symbol Power_Management:AUIPS2041L
- removed R1, R12, R18, R21, R4, R5, R8, R9: DNP, Resistor_SMD:R_2512_6332Metric, symbol Device:R
- removed R10, R11, R19, R2, R20, R7: 22, hellen-one-common:R0603, symbol hellen-one-common:Res
- removed R13, R14: DNP, Resistor_SMD:R_0402_1005Metric, symbol hellen-one-common:Res
- removed R15: 100k, Resistor_SMD:R_0402_1005Metric, symbol Device:R
- removed R16: 100, Resistor_SMD:R_0402_1005Metric, symbol Device:R
- removed R17, R24, R25: 10k, Resistor_SMD:R_0402_1005Metric, symbol Device:R
- removed R22, R23: 2.7k, hellen-one-common:R0603, symbol hellen-one-common:Res
- removed R26, R27, R28: 680k, hellen-one-common:R0603, symbol hellen-one-common:Res
- removed R29, R30: DNP, hellen-one-common:R0603, symbol hellen-one-common:Res
- removed R31: 1k6, Resistor_SMD:R_0402_1005Metric, symbol Device:R
- removed R32: 750R, Resistor_SMD:R_0402_1005Metric, symbol Device:R
- removed R33, R34, R35: 5k1, Resistor_SMD:R_0402_1005Metric, symbol Device:R
- removed R36: 20k, Resistor_SMD:R_0402_1005Metric, symbol Device:R
- removed R37: 4.7k, Resistor_SMD:R_0402_1005Metric, symbol Device:R
- removed RN1, RN2: 4.7k, Resistor_SMD:R_Array_Concave_4x0603, symbol Device:R_Pack04
- removed RN3, RN4: 1k, Resistor_SMD:R_Array_Concave_4x0603, symbol Device:R_Pack04
- removed SW1, SW2: Button_SPST, hellen-one-common:SMD-2_2.9x3.9x1.7, symbol hellen-one-common:Button_SPST
- removed TP1, TP2, TP3, TP4: TestPoint, TestPoint:TestPoint_Pad_D1.0mm, symbol Connector:TestPoint
- removed U1: TLS115_SOIC, hellen-one-common:PG-DSO-8-43, symbol hellen-one-common:TLS115
- removed U2: TLS115_SON, Package_SON:HVSON-8-1EP_3x3mm_P0.65mm_EP1.6x2.4mm, symbol hellen-one-common:TLS115
- removed U3: MCP6002-xSN, Package_SO:SOIC-8_3.9x4.9mm_P1.27mm, symbol Amplifier_Operational:MCP6002-xSN
- removed U4: L6205PD, hellen-one-common:SO20POWER, symbol hellen-one-common:L6205PD
- removed U5: MPX4_MAP, hellen-one-common:MPXH6400A-SSOP8, symbol hellen-one-common:MPX4_MAP
- removed U6: MPXA6115A, Package_SO:SSO-8_6.8x5.9mm_P1.27mm_Clearance7mm, symbol Sensor_Pressure:MPXA6115A
- removed U7: LIS2DW12TR, hellen-one-common:LGA-12_2x2mm_P0.5mm, symbol hellen-one-common:LIS2DW12TR
- removed U8: LPS25HB, Package_LGA:ST_HLGA-10_2.5x2.5mm_P0.6mm_LayoutBorder3x2y, symbol Sensor_Pressure:LPS25HB
- removed VIN1: VIN9, Connector_PinHeader_1.00mm:PinHeader_1x01_P1.00mm_Vertical, symbol Connector_Generic:Conn_01x01
- removed VIN10: VIN16, Connector_PinHeader_1.00mm:PinHeader_1x01_P1.00mm_Vertical, symbol Connector_Generic:Conn_01x01
- removed VIN11: VIN17, Connector_PinHeader_1.00mm:PinHeader_1x01_P1.00mm_Vertical, symbol Connector_Generic:Conn_01x01
- removed VIN2, VIN3, VIN4, VIN5, VIN6, VIN7, VIN8: VIN8, Connector_PinHeader_1.00mm:PinHeader_1x01_P1.00mm_Vertical, symbol Connector_Generic:Conn_01x01
- removed VIN9: VIN10, Connector_PinHeader_1.00mm:PinHeader_1x01_P1.00mm_Vertical, symbol Connector_Generic:Conn_01x01
- removed VOUT1, VOUT10, VOUT11, VOUT12, VOUT14, VOUT15, VOUT16, VOUT17, VOUT19, VOUT2, VOUT20, VOUT21, VOUT22, VOUT23, VOUT24, VOUT25, VOUT26, VOUT3, VOUT4, VOUT5, VOUT6, VOUT7, VOUT8, VOUT9: VOUT4, Connector_PinHeader_1.00mm:PinHeader_1x01_P1.00mm_Vertical, symbol Connector_Generic:Conn_01x01
- removed VOUT13: VOUT5, Connector_PinHeader_1.00mm:PinHeader_1x01_P1.00mm_Vertical, symbol Connector_Generic:Conn_01x01
- removed VOUT18: VOUT6, Connector_PinHeader_1.00mm:PinHeader_1x01_P1.00mm_Vertical, symbol Connector_Generic:Conn_01x01
- removed cr1, cr10, cr11, cr12, cr13, cr14, cr15, cr16, cr17, cr18, cr19, cr2, cr20, cr21, cr22, cr3, cr4, cr5, cr6, cr7, cr8, cr9: cr, Connector_PinHeader_1.00mm:PinHeader_1x01_P1.00mm_Vertical, symbol Connector_Generic:Conn_01x01
- added BT1: CR1220, kicad6-libraries:CR1220-2, symbol Device:Battery_Cell
- added C3: 100n, hellen-one-common:C0603, symbol hellen-one-common:Cap
- added D10: 1N4148WS, hellen-one-common:SOD-323, symbol hellen-one-common:1N4148WS
- added F6 (x4): 12H1500D, hellen-one-common:PAD-1206-PAD, symbol hellen-one-common:Fuse-Pad-Pad
- added G1: RUSEFI_LOGO, kicad6-libraries:rusefi_logo, symbol rusefi_logo:RUSEFI_LOGO
- added G2: LOGO, hellen-one-common:LOGO, symbol hellen-one-common:LOGO
- added H3, H4: M3, MountingHole:MountingHole_3.2mm_M3_Pad_Via, symbol Mechanical:MountingHole
- added J1: USB_C, kicad6-libraries:USB_C, symbol misc:USB_C
- added J1: USB_B_Mini, hellen-one-common:USB-MINI-B-VERTICAL, symbol hellen-one-common:USB_B_Mini
- added J10: Conn_02x08_Odd_Even, Connector_PinHeader_2.54mm:PinHeader_2x08_P2.54mm_Vertical, symbol Connector_Generic:Conn_02x08_Odd_Even
- added J17: Conn_01x06, Connector_PinHeader_2.54mm:PinHeader_1x06_P2.54mm_Vertical, symbol Connector_Generic:Conn_01x06
- added J2: Conn_02x10_Odd_Even, Connector_PinHeader_2.54mm:PinHeader_2x10_P2.54mm_Vertical, symbol Connector_Generic:Conn_02x10_Odd_Even
- added J3: Conn_02x03_Odd_Even, Connector_PinHeader_2.54mm:PinHeader_2x03_P2.54mm_Vertical, symbol Connector_Generic:Conn_02x03_Odd_Even
- added J4: Conn_02x04_Odd_Even, Connector_PinHeader_2.54mm:PinHeader_2x04_P2.54mm_Vertical, symbol Connector_Generic:Conn_02x04_Odd_Even
- added J5: Conn_01x05_Male, Connector_Molex:Molex_SPOX_5267-05A_1x05_P2.50mm_Vertical, symbol Connector:Conn_01x05_Pin
- added J5: Conn_02x09_Odd_Even, Connector_PinHeader_2.54mm:PinHeader_2x09_P2.54mm_Vertical, symbol Connector_Generic:Conn_02x09_Odd_Even
- added M1: Module-power_12and5V-0.2, hellen-one-power_12and5V-0.2:power_12and5V, symbol hellen-one-power_12and5V:Module-power_12and5V-0.2
- added M3: Module-knock-0.2, hellen-one-knock-0.2:knock, symbol hellen-one-knock-0.2:Module-knock-0.2
- added M3: Module-vr-discrete-0.5, hellen-one-vr-discrete-0.5:vr-discrete, symbol hellen-one-vr-discrete-0.5:Module-vr-discrete-0.5
- added M4: Module-vr-max9924-0.1, hellen-one-vr-max9924-0.1:vr-max9924, symbol vr-max9924:Module-vr-max9924-0.1
- added M5: Module-wbo-0.5, hellen-one-wbo-0.5:wbo, symbol hellen-one-wbo-0.5:Module-wbo-0.5
- added M6: Module:mega-mcu100/0.3, hellen-one-mega-mcu100-0.3:mega-mcu100, symbol hellen-one-mega-mcu100-0.3:Module{colon}mega-mcu100/0.3
- added M7: Module-can-0.1, hellen-one-can-0.1:can, symbol hellen-one-can-0.1:Module-can-0.1
- added P1, P2, P3, P4, P7, P8: Pad, hellen-one-common:PAD-TH, symbol hellen-one-common:Pad
- added R30: 33k, hellen-one-common:R0603, symbol hellen-one-common:Res
- added R30 (x2): 0, hellen-one-common:R0603, symbol hellen-one-common:Res
- added R30: 6.8k, hellen-one-common:R0603, symbol hellen-one-common:Res
- added R30: 4.7k, hellen-one-common:R0603, symbol hellen-one-common:Res
- added R38 (x3): 10k, hellen-one-common:R0805, symbol hellen-one-common:Res
- added R38, R39, R41: DNP, hellen-one-common:R0805, symbol hellen-one-common:Res
- added R4: Jumper-Pad-Pad, hellen-one-common:PAD-0805-PAD, symbol hellen-one-common:Jumper-Pad-Pad
- added U4: JDY-33, kicad6-libraries:JDY-33, symbol JDY-33:JDY-33
- H1, H2: value MountingHole -> M3; footprint MountingHole:MountingHole_4.3mm_M4_DIN965 -> MountingHole:MountingHole_3.2mm_M3_Pad_Via
- R3, R6: value 22 -> 5.6k; LCSC C23345 -> C23189
Connections:
- net +12V: now also F6.1, F6.1, F6.1, J4.7 (Pin_7), R30.2
- net +12V_RAW: now also G3.10, G3.15, G3.5, F6.2, J3.2 (Pin_2), M1.V1 (V12_PERM), M1.V3 (V12_RAW)
- net +5V: now also M1.E4 (V5), M6.N22 (VCC)
- net +5VA: now also G3.14, G3.4, G3.9, M3.E1 (V5A), M3.E4 (V5_IN), M4.E4 (V5_IN), M5.W1 (V5_IN), M6.E1 (V5A_SWITCHABLE), M6.W2 (V5A_SWITCHABLE), M7.V1 (V5), R38.2, R39.2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
- net +5VP: now also J10.6 (Pin_6), J10.8 (Pin_8), J2.2 (Pin_2), J2.4 (Pin_4), M1.V4 (5VP), R30.1
- net CAN+: now also J10.14 (Pin_14), M5.W4 (CANH), M6.W11 (CANH)
- net CAN-: now also J10.16 (Pin_16), M5.W3 (CANL), M6.W12 (CANL)
- net GND: now also G3.1, G3.11, G3.12, G3.2, G3.6, G3.7, R3.1, R6.1, BT1.2 (-), C3.1, J1.5 (GND), J1.6 (Shield)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
- net IGN1: now also M6.W10 (IGN1_(PC13))
- net IGN2: now also M6.W9 (IGN2_(PE5))
- net IGN3: now also M6.W8 (IGN3_(PE4))
- net IGN4: now also M6.W7 (IGN4_(PE3))
- net IGN5: now also M6.W6 (IGN5_(PE2))
- net IGN6: now also M6.W5 (IGN6_(PB8))
- net INJ1: now also M6.E17 (OUT_INJ1_(PD3))
- net INJ2: now also M6.E16 (OUT_INJ2_(PA9))
- net INJ3: now also M6.E15 (OUT_INJ3_(PD11))
- net INJ4: now also M6.E14 (OUT_INJ4_(PD10))
- net INJ5: now also M6.E13 (OUT_INJ5_(PD2))
- net INJ6: now also M6.E12 (OUT_INJ6_(PA8))
- net IN_CLT: now also J10.15 (Pin_15), M6.S21 (IN_CLT_(PC2))
- net IN_IAT: now also J10.13 (Pin_13), M6.S20 (IN_IAT_(PC3))
- net IN_PPS1: now also J10.12 (Pin_12), M6.S19 (IN_PPS_(PA3))
- net IN_PPS2: now also J2.8 (Pin_8), M6.S8 (IN_AUX2_(PC4/PE9))
- net IN_TPS2: now also J2.7 (Pin_7), M6.S9 (IN_AUX1_(PB0))
- net IN_VIGN: now also F6.2, M1.V2 (IN_VIGN)
- net OUT_IGN1: now also J5.11 (Pin_11)
- net OUT_IGN2: now also J5.9 (Pin_9)
- net OUT_IGN3: now also J5.5 (Pin_5)
- net OUT_IGN4: now also J5.3 (Pin_3); no longer R6.2
- net OUT_IGN5: now also J5.7 (Pin_7); no longer R3.2
- net OUT_IGN6: now also J5.1 (Pin_1)
- net OUT_INJ1: now also J5.12 (Pin_12)
- net OUT_INJ2: now also J5.10 (Pin_10)
- net OUT_INJ3: now also J5.8 (Pin_8)
- new net: J1.A5 (CC1), R3.2
- new net: J1.B5 (CC2), R6.2
- new net: M1.E6 (PG_5VP), R4.1
- new net: M6.N13 (UART2_TX_(PD5)), P8.1 (Pin_1), U4.2 (RXD)
- new net: M6.E6 (SPI2_CS_/_CAN2_RX_(PB12)), M7.V6 (CAN_RX)
- new net: M6.E7 (SPI2_SCK_/_CAN2_TX_(PB13)), M7.V5 (CAN_TX)
- new net: M6.N14 (UART2_RX_(PD6)), P7.1 (Pin_1), U4.1 (TXD)
- new net: M6.N14a (LED_GREEN), P4.1 (Pin_1)
- new net: M6.N14b (LED_YELLOW), P3.1 (Pin_1)
- new net: M5.J1 (SEL1), M5.J_GND1 (PULL_DOWN1)
- new net: J17.5 (Pin_5), M5.W5 (nReset)
- new net: J17.4 (Pin_4), M5.W6 (SWDIO)
- new net: J17.2 (Pin_2), M5.W7 (SWCLK)
- new net: J17.1 (Pin_1), M5.W8 (V33_OUT)
- new net: BT1.1 (+), D10.2 (A)
- new net: M7.S1 (CANL), P1.1 (Pin_1)
- new net: M7.S2 (CANH), P2.1 (Pin_1)
- new net +3.3V: M6.N21 (V33)
- new net 12V_KEY: F6.1, J4.5 (Pin_5)
- new net ADC3: M6.S15 (IN_KNOCK_(PA2)), R30.2, R30.2
- new net DC Driver 1/PWR: F6.2
- new net DC Driver 2/PWR: F6.2
- new net DC1_DIR: M6.E21 (OUT_PWM4_(PC8))
- new net DC1_DIS: M6.E8 (SPI2_MISO_(PB14))
- new net DC1_PWM: M6.E20 (OUT_PWM3_(PC7))
- new net DC2_DIR: M6.E9 (SPI2_MOSI_(PB15))
- new net DC2_DIS: M6.N4 (USBID_(PA10))
- new net DC2_PWM: M6.E22 (OUT_PWM5_(PC9))
- new net EGT+: J2.20 (Pin_20)
- new net EGT-: J2.19 (Pin_19)
- new net EGT/SPI_CS: M6.N9 (SPI3_CS_(PA15))
- new net EGT/SPI_SCK: M6.N10 (SPI3_SCK_(PC10))
- new net EGT/SPI_SO: M6.N11 (SPI3_MISO_(PC11))
- new net GNDA: J10.5 (Pin_5), J10.7 (Pin_7), J2.1 (Pin_1), J2.3 (Pin_3), J2.5 (Pin_5), M6.W1 (GNDA), R38.1, R38.1, R38.1
- new net INTERNAL_MAP: M6.S12 (IN_MAP2_(PC1))
- new net IN_AUX1: J10.2 (Pin_2), M6.S11 (IN_O2S_/_CAN_WAKEUP_(PA0))
- new net IN_AUX2: J2.6 (Pin_6), M6.S10 (IN_O2S2_(PA1))
- new net IN_AUX3: J2.9 (Pin_9), M6.S7 (IN_AUX3_(PA7))
- new net IN_BUTTON1: J10.4 (Pin_4), M6.S14 (IN_CRANK_(PB1)), R38.1, R38.2
- new net IN_BUTTON2: J10.3 (Pin_3), M6.S16 (IN_CAM_(PA6)), R38.2, R39.1
- new net IN_BUTTON3: J2.18 (Pin_18), M6.S1 (IN_D4_(PE15)), R38.2, R41.1
- new net IN_FLEX: J10.10 (Pin_10), M6.S17 (IN_VSS_(PE11))
- new net IN_HALL1: J2.10 (Pin_10), M6.S4 (IN_D1_(PE12))
- new net IN_HALL2: J2.12 (Pin_12), M6.S3 (IN_D2_(PE13))
- new net IN_HALL3: J2.14 (Pin_14), M6.S2 (IN_D3_(PE14))
- new net IN_KNOCK: M3.E3 (OUT_KNOCK), R30.1
- new net IN_KNOCK_RAW: J10.11 (Pin_11), M3.W1 (IN_KNOCK)
- new net IN_MAP: J10.1 (Pin_1), M6.S13 (IN_MAP1_(PC0))
- new net IN_TPS1: J10.9 (Pin_9), M6.S18 (IN_TPS_(PA4))
- new net IN_VMAIN: M6.S6 (IN_AUX4_(PC5)), R30.1, R30.2
- new net LS1: M6.E11 (OUT_INJ7_(PD15))
- new net LS2: M6.E10 (OUT_INJ8_(PD12))
- new net LS3: M6.E18 (OUT_PWM1_(PD13))
- new net LS4: M6.E19 (OUT_PWM2_(PC6))
- new net LS_HOT1: M6.W4 (IGN7_(PB9))
- new net LS_HOT2: M6.W3 (IGN8_(PE6))
- new net OUT_DC1+: J4.1 (Pin_1)
- new net OUT_DC1-: J4.2 (Pin_2)
- new net OUT_DC2+: J4.3 (Pin_3)
- new net OUT_DC2-: J4.4 (Pin_4)
- new net OUT_LS1: J5.14 (Pin_14)
- new net OUT_LS2: J5.17 (Pin_17)
- new net OUT_LS3: J5.15 (Pin_15)
- new net OUT_LS4: J5.13 (Pin_13)
- new net OUT_LS_HOT1: J5.18 (Pin_18)
- new net OUT_LS_HOT2: J5.16 (Pin_16)
- new net PG_5VP: M6.N12 (SPI3_MOSI_(PC12)), R4.2
- new net PWR_EN: M1.E5 (EN_5VP), M6.N20 (OUT_PWR_EN_(PE10))
- new net USB+: J1.3 (D+), J1.A6 (D+), J1.B6 (D+), J5.3 (Pin_3), M6.N3 (USBP_(PA12))
- new net USB-: J1.2 (D-), J1.A7 (D-), J1.B7 (D-), J5.2 (Pin_2), M6.N2 (USBM_(PA11))
- new net VR_DISCRETE: M3.E3 (OUT), M6.N18 (UART8_RX_(PE0))
- new net VR_DISCRETE+: J2.15 (Pin_15), M3.W2 (VR+)
- new net VR_DISCRETE-: J2.17 (Pin_17), M3.W1 (VR-)
- new net VR_DISCRETE_A: M3.E2 (OUT_A), R30.1
- new net VR_DISCRETE_THR: M3.E1 (Thresh_IN), M6.E23 (OUT_PWM6_(PD14))
- new net VR_MAX9924: M4.E3 (OUT), M6.N19 (UART8_TX_(PE1))
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Other:
- added sheet DC Driver 1 (DC_MOTOR_0.1.kicad_sch)
- added sheet DC Driver 2 (DC_MOTOR_0.1.kicad_sch)
- added sheet EGT (egt.kicad_sch)
- added sheet Ignition (IGN6.kicad_sch)
- added sheet Injector (INJ6.kicad_sch)
- added sheet LS (LS4.kicad_sch)
- added sheet LS HOT (LS_HOT.kicad_sch)
- added sheet MAP (MAP.kicad_sch)
- note added: "3.5A MAX Always hot capable"
- note added: "3.5A MAX Solenoid load capable"
- note added: "A"
- note added: "B"
- note added: "Bluetooth Module"
- note added: "C"
- note added: "Configurable "BUTTON" pulls"
- note added: "D"
- note added: "DC Motor"
- note added: "E"
- note added: "Install a 4.7 kOhm R1 resistor for using VR2- as a hall sensor input"
- note added: "LS & HS outputs"
- note added: "Move the resistor from position R143 to R145 to enable the CAN WAKEUP function. The AUX1 analog input will be unavailable."
- note added: "Move the resistor from position R6 to R5 to use ADC3 for receiving the analog signal VR-DISCRETE instead of the knock signal"
- note added: "Pin 8 may be used for shielding VR signals"
- note added: "Pin Name Recommended function B8 OUT_LS_HOT2 Fan Relay B9 OUT_LS_HOT1 Main Relay B16 OUT_LS4 Fuel Pump Replay B18 OUT_LS2 Idle Air Valve C8 GND VR Shield C16 IN_AUX3 Fuel Pressure D10 IN_BUTTON2 A/C Request"
- note removed: "1 | Fuel pump 2 | ICV 3 | Inj 5 4 | Inj 6 5 | Inj 4 6 | GND 7 | VVT Solenoid | Inj7 8 | 9 | X 10 | X 11 | NC 12 | NC 13 | NC 14 | GND | MAF gnd 15 | GND 16 | IN CRANK+ 17 | IN CAM 18 | NC 19 | NC 20 | USB_D+ 21 | USB_D- 22 | COIL 7 23 | COIL 4 24 | COIL 6 25 | COIL 5 26 | V12_PERM 27 | OUT_MAIN 28 | GND 29 | OUT IDLE 30 | NC 31 | INJ 3 32 | INJ 2 33 | INJ 1 34 | GND 35 | INJ 8 36 | EVAP 37 | 38 |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"
- note removed: "Accelerometer"
- note removed: "Baro"
- note removed: "C540240"
- note removed: "C540241"
- note removed: "C540242"
- note removed: "C540243"
- note removed: "ETB Drive-by-wire motor connector"
- note removed: "Electronic Throttle Body/ETB"
- note removed: "Internal pullups"
- note removed: "LEDs"
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
Commit message: attempt from other user
Parts:
- removed BT1: CR1220, kicad6-libraries:CR1220-2, symbol Device:Battery_Cell
- removed C3: 100n, hellen-one-common:C0603, symbol hellen-one-common:Cap
- removed D10: 1N4148WS, hellen-one-common:SOD-323, symbol hellen-one-common:1N4148WS
- removed F6 (x4): 12H1500D, hellen-one-common:PAD-1206-PAD, symbol hellen-one-common:Fuse-Pad-Pad
- removed G1: RUSEFI_LOGO, kicad6-libraries:rusefi_logo, symbol rusefi_logo:RUSEFI_LOGO
- removed G2: LOGO, hellen-one-common:LOGO, symbol hellen-one-common:LOGO
- removed H3, H4: M3, MountingHole:MountingHole_3.2mm_M3_Pad_Via, symbol Mechanical:MountingHole
- removed J1: USB_C, kicad6-libraries:USB_C, symbol misc:USB_C
- removed J1: USB_B_Mini, hellen-one-common:USB-MINI-B-VERTICAL, symbol hellen-one-common:USB_B_Mini
- removed J10: Conn_02x08_Odd_Even, Connector_PinHeader_2.54mm:PinHeader_2x08_P2.54mm_Vertical, symbol Connector_Generic:Conn_02x08_Odd_Even
- removed J17: Conn_01x06, Connector_PinHeader_2.54mm:PinHeader_1x06_P2.54mm_Vertical, symbol Connector_Generic:Conn_01x06
- removed J2: Conn_02x10_Odd_Even, Connector_PinHeader_2.54mm:PinHeader_2x10_P2.54mm_Vertical, symbol Connector_Generic:Conn_02x10_Odd_Even
- removed J3: Conn_02x03_Odd_Even, Connector_PinHeader_2.54mm:PinHeader_2x03_P2.54mm_Vertical, symbol Connector_Generic:Conn_02x03_Odd_Even
- removed J4: Conn_02x04_Odd_Even, Connector_PinHeader_2.54mm:PinHeader_2x04_P2.54mm_Vertical, symbol Connector_Generic:Conn_02x04_Odd_Even
- removed J5: Conn_01x05_Male, Connector_Molex:Molex_SPOX_5267-05A_1x05_P2.50mm_Vertical, symbol Connector:Conn_01x05_Pin
- removed J5: Conn_02x09_Odd_Even, Connector_PinHeader_2.54mm:PinHeader_2x09_P2.54mm_Vertical, symbol Connector_Generic:Conn_02x09_Odd_Even
- removed M1: Module-power_12and5V-0.2, hellen-one-power_12and5V-0.2:power_12and5V, symbol hellen-one-power_12and5V:Module-power_12and5V-0.2
- removed M3: Module-knock-0.2, hellen-one-knock-0.2:knock, symbol hellen-one-knock-0.2:Module-knock-0.2
- removed M3: Module-vr-discrete-0.5, hellen-one-vr-discrete-0.5:vr-discrete, symbol hellen-one-vr-discrete-0.5:Module-vr-discrete-0.5
- removed M4: Module-vr-max9924-0.1, hellen-one-vr-max9924-0.1:vr-max9924, symbol vr-max9924:Module-vr-max9924-0.1
- removed M5: Module-wbo-0.5, hellen-one-wbo-0.5:wbo, symbol hellen-one-wbo-0.5:Module-wbo-0.5
- removed M6: Module:mega-mcu100/0.3, hellen-one-mega-mcu100-0.3:mega-mcu100, symbol hellen-one-mega-mcu100-0.3:Module{colon}mega-mcu100/0.3
- removed M7: Module-can-0.1, hellen-one-can-0.1:can, symbol hellen-one-can-0.1:Module-can-0.1
- removed P1, P2, P3, P4, P7, P8: Pad, hellen-one-common:PAD-TH, symbol hellen-one-common:Pad
- removed R30: 33k, hellen-one-common:R0603, symbol hellen-one-common:Res
- removed R30 (x2): 0, hellen-one-common:R0603, symbol hellen-one-common:Res
- removed R30: 6.8k, hellen-one-common:R0603, symbol hellen-one-common:Res
- removed R30: 4.7k, hellen-one-common:R0603, symbol hellen-one-common:Res
- removed R38 (x3): 10k, hellen-one-common:R0805, symbol hellen-one-common:Res
- removed R38, R39, R41: DNP, hellen-one-common:R0805, symbol hellen-one-common:Res
- removed R4: Jumper-Pad-Pad, hellen-one-common:PAD-0805-PAD, symbol hellen-one-common:Jumper-Pad-Pad
- removed U4: JDY-33, kicad6-libraries:JDY-33, symbol JDY-33:JDY-33
- added BT1: BATTERY_CR2032, Battery:BatteryHolder_Keystone_1060_1x2032, symbol art-electro-power:BATTERY_CR2032
- added C1, C2: 1u, hellen-one-common:C0603, symbol hellen-one-common:Cap
- added C10: 10nF, Capacitor_SMD:C_0402_1005Metric, symbol Device:C
- added C11, C12, C13, C15, C18, C20, C5, C6, C7, C9: 10u, Capacitor_SMD:C_0603_1608Metric, symbol Device:C
- added C14: 220nF, Capacitor_SMD:C_0402_1005Metric, symbol Device:C
- added C16, C17, C19, C21, C23, C3, C4: 100nF, Capacitor_SMD:C_0402_1005Metric, symbol Device:C
- added C22: 100n, hellen-one-common:C0603, symbol hellen-one-common:Cap
- added C8: 5.6nF, Capacitor_SMD:C_0402_1005Metric, symbol Device:C
- added D1, D2: B5819W, Diode_SMD:D_SOD-123, symbol Diode:1N4148WS
- added D10, D12, D14, D16, D18, D20, D22, D37, D39, D8: LED-RED-0603, LED_SMD:LED_0603_1608Metric, symbol Device:LED
- added D11, D13, D15, D17, D19, D21, D34, D36, D38, D40, D42, D7, D9: 1N4148WS, Diode_SMD:D_SOD-323, symbol Diode:1N4148WS
- added D23, D24, D25, D26, D27, D28, D29, D30: LED-BLUE-0603, LED_SMD:LED_0603_1608Metric, symbol Device:LED
- added D3, D4: 1N4148WS, Diode_SMD:D_SOD-323, symbol Device:D
- added D31, D32, D33, D35: LED-GREEN-0603, LED_SMD:LED_0603_1608Metric, symbol Device:LED
- added D41: LED-WHITE-0603, LED_SMD:LED_0603_1608Metric, symbol Device:LED
- added D43: 1N4148WS, hellen-one-common:SOD-323, symbol hellen-one-common:1N4148WS
- added D5, D6: B5819W, Diode_SMD:D_SOD-123, symbol hellen-one-common:1N4148WS
- added F1, F2, F3, F4, F5, F6, F7, F8: 10A, hellen-one-common:36911600000, symbol hellen-one-common:Fuse-Pad-Pad
- added G1, G2: PROTO_AREA, hellen-one-common:PROTO_AREA, symbol hellen-one-common:PROTO_AREA
- added J1: Conn_01x05, Connector_PinHeader_2.54mm:PinHeader_1x05_P2.54mm_Vertical, symbol Connector_Generic:Conn_01x05
- added J10: Conn_01x05, Connector_PinHeader_2.00mm:PinHeader_1x05_P2.00mm_Vertical, symbol Connector_Generic:Conn_01x05
- added J11: USB_B_Mini, hellen-one-common:USB-MINI-B-VERTICAL, symbol hellen-one-common:USB_B_Mini
- added J2: MiniFit, Connector_Molex:Molex_Mini-Fit_Jr_5569-02A2_2x01_P4.20mm_Horizontal, symbol Connector_Generic:Conn_01x02
- added J3: VRIN1, Connector_PinHeader_1.00mm:PinHeader_1x01_P1.00mm_Vertical, symbol Connector_Generic:Conn_01x01
- added J4: VRIN2, Connector_PinHeader_1.00mm:PinHeader_1x01_P1.00mm_Vertical, symbol Connector_Generic:Conn_01x01
- added J5: AudioJack_THR, hellen-one-common:Jack_3.5mm_PJ-3250-5A, symbol hellen-one-common:AudioJack_THR
- added J6: VROUT1, Connector_PinHeader_1.00mm:PinHeader_1x01_P1.00mm_Vertical, symbol Connector_Generic:Conn_01x01
- added J7: ETB, Connector_PinHeader_2.54mm:PinHeader_1x06_P2.54mm_Vertical, symbol Connector_Generic:Conn_01x06
- added J8: PPS, Connector_PinHeader_2.54mm:PinHeader_1x04_P2.54mm_Vertical, symbol Connector_Generic:Conn_01x04
- added J9: XH-8A, kicad6:XH-8A, symbol Connector_Generic:Conn_01x08
- added JP1, JP10, JP11, JP12, JP13, JP14, JP15, JP16, JP17, JP18, JP19, JP2, JP20, JP21, JP22, JP23, JP24, JP25, JP28, JP29, JP3, JP30, JP31, JP32, JP33, JP34, JP35, JP4, JP5, JP6, JP7, JP8, JP9: Jumper_2_Open, hellen-one-common:PAD-0805-PAD, symbol hellen-one-common:Jumper-Pad-Pad
- added JP26, JP27: Jumper_2_Open, hellen-one-common:PAD-1206-PAD, symbol hellen-one-common:Fuse-Pad-Pad
- added KNOCK_RAW1: IN_KNOCK1_RAW, Connector_PinHeader_1.00mm:PinHeader_1x01_P1.00mm_Vertical, symbol Connector_Generic:Conn_01x01
- added KNOCK_RAW2: IN_KNOCK2_RAW, Connector_PinHeader_1.00mm:PinHeader_1x01_P1.00mm_Vertical, symbol Connector_Generic:Conn_01x01
- added M1: Module-power12-0.2, hellen-one-power12-0.2:power12, symbol power12-0.2:Module-power12-0.2
- added M10: Module-sd-0.1, hellen-one-sd-0.1:sd, symbol sd-0.1:Module-sd-0.1
- added M11, M13: Module-can-0.1, hellen-one-can-0.1:can, symbol can-0.1:Module-can-0.1
- added M12: Module-wbo-0.3, hellen-one-wbo-0.3:wbo, symbol wbo-0.3:Module-wbo-0.3
- added M2: Module-power5-0.2, hellen-one-power5-0.2:power5, symbol power5-0.2:Module-power5-0.2
- added M3, M4: Module-knock-0.1, hellen-one-knock-0.1:knock, symbol knock-0.1:Module-knock-0.1
- added M5: Module-vr-0.1, hellen-one-vr-0.1:vr, symbol hellen-one-vr-0.1:Module-vr-0.1
- added M6: Module-output-0.3, hellen-one-output-0.3:output, symbol output-0.3:Module-output-0.3
- added M7: Module-input-0.1, hellen-one-input-0.1:input, symbol input-0.1:Module-input-0.1
- added M8: Module-ign8-0.2, hellen-one-ign8-0.2:ign8, symbol ign8-0.2:Module-ign8-0.2
- added M9: Module-mcu144-0.6, hellen-one-mcu-0.6:mcu, symbol mcu-0.6:Module-mcu-0.6
- added MMCU1, MMCU10, MMCU11, MMCU12, MMCU13, MMCU14, MMCU15, MMCU16, MMCU17, MMCU18, MMCU19, MMCU2, MMCU20, MMCU21, MMCU22, MMCU23, MMCU24, MMCU25, MMCU26, MMCU27, MMCU28, MMCU29, MMCU3, MMCU30, MMCU31, MMCU4, MMCU5, MMCU6, MMCU7, MMCU8, MMCU9: MMCU, Connector_PinHeader_1.00mm:PinHeader_1x01_P1.00mm_Vertical, symbol Connector_Generic:Conn_01x01
- added P1, P2, P3, P4, P5, P6: P, Connector_Pin:Pin_D1.0mm_L10.0mm, symbol Connector_Generic:Conn_01x01
- added PP1: Motronic_88pin, rusefi_lib_private:88pin_STS, symbol motronic_88pin_STS:Motronic_88pin
- added Q1, Q2, Q3, Q4, Q5, Q6, Q7, Q8: NGD8201AN, Package_TO_SOT_SMD:TO-252-2, symbol Device:Q_NIGBT_GCE
- added Q10, Q9: AUIPS2041LTR, Package_TO_SOT_SMD:SOT-223, symbol Power_Management:AUIPS2041L
- added R1, R12, R18, R21, R4, R5, R8, R9: DNP, Resistor_SMD:R_2512_6332Metric, symbol Device:R
- added R10, R11, R19, R2, R20, R7: 22, hellen-one-common:R0603, symbol hellen-one-common:Res
- added R13, R14: DNP, Resistor_SMD:R_0402_1005Metric, symbol hellen-one-common:Res
- added R15: 100k, Resistor_SMD:R_0402_1005Metric, symbol Device:R
- added R16: 100, Resistor_SMD:R_0402_1005Metric, symbol Device:R
- added R17, R24, R25: 10k, Resistor_SMD:R_0402_1005Metric, symbol Device:R
- added R22, R23: 2.7k, hellen-one-common:R0603, symbol hellen-one-common:Res
- added R26, R27, R28: 680k, hellen-one-common:R0603, symbol hellen-one-common:Res
- added R29, R30: DNP, hellen-one-common:R0603, symbol hellen-one-common:Res
- added R31: 1k6, Resistor_SMD:R_0402_1005Metric, symbol Device:R
- added R32: 750R, Resistor_SMD:R_0402_1005Metric, symbol Device:R
- added R33, R34, R35: 5k1, Resistor_SMD:R_0402_1005Metric, symbol Device:R
- added R36: 20k, Resistor_SMD:R_0402_1005Metric, symbol Device:R
- added R37: 4.7k, Resistor_SMD:R_0402_1005Metric, symbol Device:R
- added RN1, RN2: 4.7k, Resistor_SMD:R_Array_Concave_4x0603, symbol Device:R_Pack04
- added RN3, RN4: 1k, Resistor_SMD:R_Array_Concave_4x0603, symbol Device:R_Pack04
- added SW1, SW2: Button_SPST, hellen-one-common:SMD-2_2.9x3.9x1.7, symbol hellen-one-common:Button_SPST
- added TP1, TP2, TP3, TP4: TestPoint, TestPoint:TestPoint_Pad_D1.0mm, symbol Connector:TestPoint
- added U1: TLS115_SOIC, hellen-one-common:PG-DSO-8-43, symbol hellen-one-common:TLS115
- added U2: TLS115_SON, Package_SON:HVSON-8-1EP_3x3mm_P0.65mm_EP1.6x2.4mm, symbol hellen-one-common:TLS115
- added U3: MCP6002-xSN, Package_SO:SOIC-8_3.9x4.9mm_P1.27mm, symbol Amplifier_Operational:MCP6002-xSN
- added U4: L6205PD, hellen-one-common:SO20POWER, symbol hellen-one-common:L6205PD
- added U5: MPX4_MAP, hellen-one-common:MPXH6400A-SSOP8, symbol hellen-one-common:MPX4_MAP
- added U6: MPXA6115A, Package_SO:SSO-8_6.8x5.9mm_P1.27mm_Clearance7mm, symbol Sensor_Pressure:MPXA6115A
- added U7: LIS2DW12TR, hellen-one-common:LGA-12_2x2mm_P0.5mm, symbol hellen-one-common:LIS2DW12TR
- added U8: LPS25HB, Package_LGA:ST_HLGA-10_2.5x2.5mm_P0.6mm_LayoutBorder3x2y, symbol Sensor_Pressure:LPS25HB
- added VIN1: VIN9, Connector_PinHeader_1.00mm:PinHeader_1x01_P1.00mm_Vertical, symbol Connector_Generic:Conn_01x01
- added VIN10: VIN16, Connector_PinHeader_1.00mm:PinHeader_1x01_P1.00mm_Vertical, symbol Connector_Generic:Conn_01x01
- added VIN11: VIN17, Connector_PinHeader_1.00mm:PinHeader_1x01_P1.00mm_Vertical, symbol Connector_Generic:Conn_01x01
- added VIN2, VIN3, VIN4, VIN5, VIN6, VIN7, VIN8: VIN8, Connector_PinHeader_1.00mm:PinHeader_1x01_P1.00mm_Vertical, symbol Connector_Generic:Conn_01x01
- added VIN9: VIN10, Connector_PinHeader_1.00mm:PinHeader_1x01_P1.00mm_Vertical, symbol Connector_Generic:Conn_01x01
- added VOUT1, VOUT10, VOUT11, VOUT12, VOUT14, VOUT15, VOUT16, VOUT17, VOUT19, VOUT2, VOUT20, VOUT21, VOUT22, VOUT23, VOUT24, VOUT25, VOUT26, VOUT3, VOUT4, VOUT5, VOUT6, VOUT7, VOUT8, VOUT9: VOUT4, Connector_PinHeader_1.00mm:PinHeader_1x01_P1.00mm_Vertical, symbol Connector_Generic:Conn_01x01
- added VOUT13: VOUT5, Connector_PinHeader_1.00mm:PinHeader_1x01_P1.00mm_Vertical, symbol Connector_Generic:Conn_01x01
- added VOUT18: VOUT6, Connector_PinHeader_1.00mm:PinHeader_1x01_P1.00mm_Vertical, symbol Connector_Generic:Conn_01x01
- added cr1, cr10, cr11, cr12, cr13, cr14, cr15, cr16, cr17, cr18, cr19, cr2, cr20, cr21, cr22, cr3, cr4, cr5, cr6, cr7, cr8, cr9: cr, Connector_PinHeader_1.00mm:PinHeader_1x01_P1.00mm_Vertical, symbol Connector_Generic:Conn_01x01
- H1, H2: value M3 -> MountingHole; footprint MountingHole:MountingHole_3.2mm_M3_Pad_Via -> MountingHole:MountingHole_4.3mm_M4_DIN965
- R3, R6: value 5.6k -> 22; LCSC C23189 -> C23345
Connections:
- net +12V: now also D33.2 (A), D34.1 (K), M1.V1 (V12), M2.V1 (V12), TP4.1
- net +12V_RAW: now also C11.1, C12.1, C13.1, C14.1, C15.1, C16.1, C18.1, C19.1, C20.1, C7.1, C9.1, D1.1 (K)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; no longer G3.10, G3.15, G3.5
- net +5V: now also C3.1, D31.2 (A), J1.4 (Pin_4), M1.E1 (V5), M11.V1 (V5), M12.W1 (V5_IN), M13.V1 (V5), M2.V2 (V5), M5.N1 (V5), M6.W14 (V5), M7.E2 (V5), M9.S1 (V5)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
- net +5VA: now also C17.1, C4.1, M3.E1 (V5A), M4.E1 (V5A), M7.E5 (V5A), M7.J1 (PULL_V5A), M7.J17 (PULL_CAM), M7.J18 (PULL_VSS), M7.J21 (PULL_CRANK), M7.J7 (PULL_AUX4), M7.N1 (V5A), M9.S33 (V5A)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; no longer G3.14, G3.4, G3.9
- net +5VP: now also C2.2, J7.1 (Pin_1), J7.2 (Pin_2), J8.1 (Pin_1), JP28.2, U1.1 (OUT), U2.1 (OUT)
- net CAN+: now also JP33.2, M11.S2 (CANH), M13.S2 (CANH)
- net CAN-: now also JP32.2, M11.S1 (CANL), M13.S1 (CANL)
- net GND: now also BT1.2 (-), C1.1, C11.2, C12.2, C13.2, C15.2, C16.2, C17.2, C18.2, C19.2, C2.1, C20.2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; no longer G3.1, G3.11, G3.12, G3.2, G3.6, G3.7, R3.1, R6.1
- net IGN1: now also M8.V8 (IGN1), M9.W1 (OUT_IGN1)
- net IGN2: now also M8.V7 (IGN2), M9.W2 (OUT_IGN2)
- net IGN3: now also M8.V6 (IGN3), M9.W3 (OUT_IGN3)
- net IGN4: now also M8.V5 (IGN4), M9.W4 (OUT_IGN4)
- net IGN5: now also M8.V4 (IGN5), M9.W5 (OUT_IGN5)
- net IGN6: now also M8.V3 (IGN6), M9.W6 (OUT_IGN6)
- net INJ1: now also M6.W24 (INJ1), M9.E25 (OUT_INJ1)
- net INJ2: now also M6.W23 (INJ2), M9.E26 (OUT_INJ2)
- net INJ3: now also M6.W20 (INJ3), M9.E29 (OUT_INJ3)
- net INJ4: now also M6.W19 (INJ4), M9.E30 (OUT_INJ4)
- net INJ5: now also M6.W18 (INJ5), M9.E31 (OUT_INJ5)
- net INJ6: now also M6.W17 (INJ6), M9.E32 (OUT_INJ6)
- net IN_CLT: now also JP31.2, M7.S15 (IN_CLT), R22.1
- net IN_IAT: now also JP30.2, M7.S16 (IN_IAT), R23.1
- net IN_PPS1: now also J8.3 (Pin_3), M7.S24 (IN_PPS)
- net IN_PPS2: now also J8.2 (Pin_2), M7.S18 (IN_AUX2), R28.2
- net IN_TPS2: now also J7.4 (Pin_4), M7.S17 (IN_AUX1), R26.2
- net IN_VIGN: now also JP34.2, M1.V3 (IN_VIGN)
- new net: Q4.1 (G), R7.1
- new net: PP1.87, cr20.1 (Pin_1)
- new net: M7.S25 (IN_O2S2), VIN6.1 (Pin_1)
- new net: D15.1 (K), D16.2 (A), RN2.5 (R4.2)
- new net: D25.1 (K), RN4.5 (R4.2)
- new net: M9.N4 (UART8_TX), MMCU21.1 (Pin_1)
- new net: D28.1 (K), RN3.8 (R1.2)
- new net: D35.1 (K), D36.2 (A), R34.1
- new net: M6.S14 (OUT_LOW9), VOUT5.1 (Pin_1)
- new net: J6.1 (Pin_1), M5.W1 (OUT_VR2)
- new net: D39.2 (A), D40.1 (K), R36.2
- new net: Q5.1 (G), R10.1
- new net: M9.N12 (IO1), MMCU28.1 (Pin_1)
- new net: M6.S5 (OUT_SOLENOID_B2), VOUT11.1 (Pin_1)
- new net: C10.1, R16.1
- new net: D3.1 (K), D4.2 (A), R16.2
- new net: JP28.1, PP1.59
- new net: D17.1 (K), D18.2 (A), RN2.6 (R3.2)
- new net: D21.1 (K), D22.2 (A), RN2.8 (R1.2)
- new net: M9.N32 (USB1ID), MMCU24.1 (Pin_1)
- new net: Q3.1 (G), R6.1
- new net: C6.1, U3.6 (-), U3.7
- new net: C6.2, J5.R
- new net: M6.W37 (LOW8_HIGH2), VOUT14.1 (Pin_1)
- new net: M9.N13 (IO2), MMCU29.1 (Pin_1)
- new net: M9.N14 (IO3), MMCU30.1 (Pin_1)
- new net: M9.N15 (IO4), MMCU31.1 (Pin_1)
- new net: JP1.1, PP1.1
- new net: C5.1, U3.1, U3.2 (-)
- new net: C5.2, J5.T
- new net: M7.S23 (IN_RES1), VIN2.1 (Pin_1)
- new net: D41.2 (A), D42.1 (K), R37.2
- new net: PP1.11, cr1.1 (Pin_1)
- new net: PP1.13, cr3.1 (Pin_1)
- new net: D2.2 (A), JP35.2
- new net: JP2.1, PP1.3
- new net: PP1.37, cr8.1 (Pin_1)
- new net: D23.1 (K), RN3.5 (R4.2)
- new net: D27.1 (K), RN3.6 (R3.2)
- new net: D24.1 (K), RN3.7 (R2.2)
- new net: J3.1 (Pin_1), M5.E3 (IN_VR2+)
- new net: J4.1 (Pin_1), M5.E4 (IN_VR2-)
- new net: M6.W31 (SOLENOID_B1), VOUT21.1 (Pin_1)
- new net: JP29.1, PP1.73
- new net: D33.1 (K), D34.2 (A), R33.1
- new net: M9.N7 (UART2_RX), MMCU22.1 (Pin_1)
- new net: M9.N25 (SWCLK), MMCU25.1 (Pin_1)
- new net: M6.W36 (LOW12), VOUT17.1 (Pin_1)
- new net: M9.E12 (OUT_IO2), MMCU2.1 (Pin_1)
- new net: M6.S12 (OUT_LOW8_PULLUP), VOUT4.1 (Pin_1)
- new net: M6.W3 (OUT_LOW6_DIODE), VOUT2.1 (Pin_1)
- new net: JP3.1, PP1.4
- new net: JP23.1, PP1.46, cr4.1 (Pin_1)
- new net: M9.N26 (SWDIO), MMCU26.1 (Pin_1)
- new net: PP1.82, cr18.1 (Pin_1)
- new net: Q2.1 (G), R3.1
- new net: PP1.60, cr10.1 (Pin_1)
- new net: JP6.1, PP1.8
- new net: JP25.1, PP1.48
- new net: M9.S5 (IN_D3), MMCU13.1 (Pin_1)
- new net: M7.S1 (IN_SENS1), VIN8.1 (Pin_1)
- new net: JP4.1, PP1.5
- new net: M6.W27 (LOW9), VOUT15.1 (Pin_1)
- new net: M9.E20 (OUT_IO11), MMCU8.1 (Pin_1)
- new net: JP27.1, JP34.1, PP1.56
- new net: C14.2, D4.1 (K), U4.17 (VBOOT)
- new net: PP1.12, cr2.1 (Pin_1)
- new net: M7.E4 (WBO_O2S), VIN10.1 (Pin_1)
- new net: PP1.68, cr16.1 (Pin_1)
- new net: D37.1 (K), D38.2 (A), R35.1
- new net: M6.S2 (OUT_SOLENOID_A2), VOUT9.1 (Pin_1)
- new net: G2.1, G2.11, G2.6
- new net: G2.10, G2.15, G2.5
- new net: G2.12, G2.2, G2.7
- new net: G2.13, G2.3, G2.8
- new net: G2.14, G2.4, G2.9
- new net: JP11.1, PP1.21
- new net: PP1.66, cr14.1 (Pin_1)
- new net: M7.S9 (IN_O2S), VIN5.1 (Pin_1)
- new net: M6.W39 (LOW7_HIGH1), VOUT26.1 (Pin_1)
- new net: M9.E9 (OUT_IO6), MMCU4.1 (Pin_1)
- new net: PP1.18, cr5.1 (Pin_1)
- new net: JP21.1, PP1.42
- new net: M9.E10 (OUT_IO10), MMCU7.1 (Pin_1)
- new net: M9.E11 (OUT_IO9), MMCU6.1 (Pin_1)
- new net: M9.E13 (OUT_IO12), MMCU9.1 (Pin_1)
- new net: M9.E16 (OUT_PWM4), MMCU1.1 (Pin_1)
- new net: M9.E22 (OUT_IO8), MMCU5.1 (Pin_1)
- new net: M9.E23 (OUT_IO4), MMCU3.1 (Pin_1)
- new net: M9.E24 (OUT_IO13), MMCU10.1 (Pin_1)
- new net: BT1.1 (+), D43.2 (A)
- new net: M9.S6 (IN_D4), MMCU14.1 (Pin_1)
- new net: C8.1, R15.1, U4.16 (ENB), U4.5 (ENA)
- new net: C10.2, U4.4 (VCP)
- new net: JP9.1, PP1.17
- new net: M6.S1 (OUT_SOLENOID_A1), VOUT8.1 (Pin_1)
- new net: M6.S10 (OUT_LOW11), VOUT6.1 (Pin_1)
- new net: M6.S13 (OUT_LOW12), VOUT7.1 (Pin_1)
- new net: M6.S4 (OUT_SOLENOID_B1), VOUT10.1 (Pin_1)
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Other:
- removed sheet DC Driver 1
- removed sheet DC Driver 2
- removed sheet EGT
- removed sheet Ignition
- removed sheet Injector
- removed sheet LS
- removed sheet LS HOT
- removed sheet MAP
- note added: "1 | Fuel pump 2 | ICV 3 | Inj 5 4 | Inj 6 5 | Inj 4 6 | GND 7 | VVT Solenoid | Inj7 8 | 9 | X 10 | X 11 | NC 12 | NC 13 | NC 14 | GND | MAF gnd 15 | GND 16 | IN CRANK+ 17 | IN CAM 18 | NC 19 | NC 20 | USB_D+ 21 | USB_D- 22 | COIL 7 23 | COIL 4 24 | COIL 6 25 | COIL 5 26 | V12_PERM 27 | OUT_MAIN 28 | GND 29 | OUT IDLE 30 | NC 31 | INJ 3 32 | INJ 2 33 | INJ 1 34 | GND 35 | INJ 8 36 | EVAP 37 | 38 |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"
- note added: "Accelerometer"
- note added: "Baro"
- note added: "C540240"
- note added: "C540241"
- note added: "C540242"
- note added: "C540243"
- note added: "ETB Drive-by-wire motor connector"
- note added: "Electronic Throttle Body/ETB"
- note added: "Internal pullups"
- note added: "LEDs"
- note added: "Ouputs"
- note added: "Protected 5V analog power supply"
- note added: "SOIC-8"
- note added: "TSON-10"
- note added: "VVT_AV7"
- note removed: "3.5A MAX Always hot capable"
- note removed: "3.5A MAX Solenoid load capable"
- note removed: "A"
- note removed: "B"
- note removed: "Bluetooth Module"
- note removed: "C"
- note removed: "Configurable "BUTTON" pulls"
- note removed: "D"
- note removed: "DC Motor"
- note removed: "E"
- note removed: "Install a 4.7 kOhm R1 resistor for using VR2- as a hall sensor input"
- note removed: "LS & HS outputs"
- note removed: "Move the resistor from position R143 to R145 to enable the CAN WAKEUP function. The AUX1 analog input will be unavailable."
- note removed: "Move the resistor from position R6 to R5 to use ADC3 for receiving the analog signal VR-DISCRETE instead of the knock signal"
- note removed: "Pin 8 may be used for shielding VR signals"
- note removed: "Pin Name Recommended function B8 OUT_LS_HOT2 Fan Relay B9 OUT_LS_HOT1 Main Relay B16 OUT_LS4 Fuel Pump Replay B18 OUT_LS2 Idle Air Valve C8 GND VR Shield C16 IN_AUX3 Fuel Pressure D10 IN_BUTTON2 A/C Request"
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